Commit message: Update

File: xrm_sensor_kit_description/urdf/sensor_kit.xacro (robot description, xacro)
@@ -29,33 +29,3 @@
       />
     </xacro:VLP-16>
-    <!-- camera -->
-    <xacro:monocular_camera_macro
-      name="camera0/camera"
-      parent="sensor_kit_base_link"
-      namespace=""
-      x="${calibration['sensor_kit_base_link']['camera0/camera_link']['x']}"
-      y="${calibration['sensor_kit_base_link']['camera0/camera_link']['y']}"
-      z="${calibration['sensor_kit_base_link']['camera0/camera_link']['z']}"
-      roll="${calibration['sensor_kit_base_link']['camera0/camera_link']['roll']}"
-      pitch="${calibration['sensor_kit_base_link']['camera0/camera_link']['pitch']}"
-      yaw="${calibration['sensor_kit_base_link']['camera0/camera_link']['yaw']}"
-      fps="30"
-      width="1920"
-      height="1080"
-      fov="1.3"
-    />
-    <!-- imu -->
-    <xacro:imu_macro
-      name="imu"
-      parent="sensor_kit_base_link"
-      namespace=""
-      x="${calibration['sensor_kit_base_link']['imu_link']['x']}"
-      y="${calibration['sensor_kit_base_link']['imu_link']['y']}"
-      z="${calibration['sensor_kit_base_link']['imu_link']['z']}"
-      roll="${calibration['sensor_kit_base_link']['imu_link']['roll']}"
-      pitch="${calibration['sensor_kit_base_link']['imu_link']['pitch']}"
-      yaw="${calibration['sensor_kit_base_link']['imu_link']['yaw']}"
-      fps="100"
-    />
-  </xacro:macro>
 </robot>

Commit message: Update sensor_kit.xacro

File: xrm_sensor_kit_description/urdf/sensor_kit.xacro (robot description, xacro)
@@ -3,6 +3,4 @@
   <xacro:macro name="sensor_kit_macro" params="parent x y z roll pitch yaw">
     <xacro:include filename="$(find velodyne_description)/urdf/VLP-16.urdf.xacro"/>
-    <xacro:include filename="$(find camera_description)/urdf/monocular_camera.xacro"/>
-    <xacro:include filename="$(find imu_description)/urdf/imu.xacro"/>
     <xacro:arg name="gpu" default="false"/>
     <xacro:arg name="config_dir" default="$(find xrm_sensor_kit_description)/config"/>
@@ -29,3 +27,4 @@
       />
     </xacro:VLP-16>
+  </xacro:macro>
 </robot>
